File: pcb/brick_lamp.kicad_pcb (KiCad board)
At the start: 2 copper layers, 25.4 x 20.3 mm, 11 parts, among them J1 LED_24V_OUT, J2 24V_IN, J3 DEBUG, J4 DEBUG, Q1 CSD17302Q5A, U2 MCP1799x-330xxTT, U3 ATtiny85V-10S

Commit message: Cleanup the layout and schematic
Parts:
- moved C2 2.01 mm to (130.8, 91.8)
Routing:
- net Net-(J1-Pin_1): track 8.83 -> 8.19 mm
- net GND: vias 38 -> 42
Other:
- board size 25.4 x 20.3 mm -> 26.7 x 21 mm
